File: Odroid Headphone Hat.brd (EAGLE design)
At the start: 65.7 x 12.9 mm, 20 parts, among them X1 1501_03, X2 1501_03

Commit message: A few tweeks
Routing:
- net GND: track 107.0 -> 101.8 mm
- net XSMT: track 12.4 -> 10.4 mm
Other:
- board text added: "(c)2018 Dr A!"
- board text removed: "(c)2019 Dr A!"
Changed lines of the file:
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@@
 <text x="40.726359375" y="0.47751875" size="1.016" layer="21" font="vector">odroid-go headphone hat v1</text>
 <text x="25.1206" y="11.47571875" size="1.016" layer="21" font="vector">backofficeshow.com</text>
-<text x="0.335278125" y="0.193040625" size="1.016" layer="21" font="vector">(c)2019 Dr A!</text>
+<text x="0.335278125" y="0.193040625" size="1.016" layer="21" font="vector">(c)2018 Dr A!</text>
 </plain>
 <attributes>
@@
 <wire x1="31.255353125" y1="10.1083625" x2="31.916803125" y2="10.1083625" width="0.254" layer="1"/>
 <wire x1="31.916803125" y1="10.1083625" x2="33.27908125" y2="11.470640625" width="0.254" layer="1"/>
-<wire x1="33.27908125" y1="11.470640625" x2="41.894759375" y2="11.470640625" width="0.254" layer="1"/>
-<wire x1="41.894759375" y1="11.470640625" x2="42.164" y2="11.2014" width="0.254" layer="1"/>
-<wire x1="42.164" y1="11.2014" x2="52.06491875" y2="11.2014" width="0.254" layer="1"/>
-<wire x1="52.06491875" y1="11.2014" x2="52.54751875" y2="10.7188" width="0.254" layer="1"/>
+<wire x1="33.27908125" y1="11.470640625" x2="43.139359375" y2="11.470640625" width="0.254" layer="1"/>
 <wire x1="52.54751875" y1="10.7188" x2="53.5296" y2="10.7188" width="0.254" layer="1"/>
 <wire x1="53.5296" y1="10.7188" x2="54.41351875" y2="9.83488125" width="0.254" layer="1"/>
+<wire x1="43.139359375" y1="11.470640625" x2="43.550840625" y2="11.0744" width="0.254" layer="1"/>
+<wire x1="43.550840625" y1="11.0744" x2="52.207159375" y2="11.0744" width="0.254" layer="1"/>
+<wire x1="52.207159375" y1="11.0744" x2="52.54751875" y2="10.7188" width="0.254" layer="1"/>
 </signal>
 <signal name="N$14">
@@
 <via x="51.08448125" y="9.80948125" extent="1-16" drill="0.6"/>
 <wire x1="51.08448125" y1="9.80948125" x2="42.636440625" y2="9.80948125" width="0.254" layer="16"/>
-<wire x1="42.636440625" y1="9.80948125" x2="42.06748125" y2="10.378440625" width="0.254" layer="16"/>
-<wire x1="42.06748125" y1="10.378440625" x2="33.975040625" y2="10.378440625" width="0.254" layer="16"/>
 <wire x1="33.975040625" y1="10.378440625" x2="33.3502" y2="9.7536" width="0.254" layer="16"/>
 <via x="33.3502" y="9.7536" extent="1-16" drill="0.6"/>
@@
 <wire x1="32.369759375" y1="8.823959375" x2="31.27095" y2="8.823959375" width="0.254" layer="1"/>
 <wire x1="31.27095" y1="8.823959375" x2="31.255353125" y2="8.8083625" width="0.254" layer="1"/>
+<wire x1="33.975040625" y1="10.378440625" x2="33.980121875" y2="10.378440625" width="0.254" layer="16"/>
+<wire x1="33.980121875" y1="10.378440625" x2="33.980121875" y2="10.388603125" width="0.254" layer="16"/>
+<wire x1="33.980121875" y1="10.388603125" x2="34.417" y2="10.82548125" width="0.254" layer="16"/>
+<wire x1="34.417" y1="10.82548125" x2="41.620440625" y2="10.82548125" width="0.254" layer="16"/>
+<wire x1="41.620440625" y1="10.82548125" x2="42.636440625" y2="9.80948125" width="0.254" layer="16"/>
 </signal>
 <signal name="N$15">
@@
 <wire x1="54.443996875" y1="7.481203125" x2="53.837840625" y2="8.087359375" width="0.254" layer="1"/>
 <wire x1="53.837840625" y1="8.087359375" x2="51.506121875" y2="8.087359375" width="0.254" layer="1"/>
-<wire x1="51.506121875" y1="8.087359375" x2="49.443640625" y2="10.149840625" width="0.254" layer="1"/>
 <wire x1="49.443640625" y1="10.149840625" x2="48.353078125" y2="10.149840625" width="0.254" layer="1"/>
 <wire x1="48.353078125" y1="10.149840625" x2="48.3362" y2="10.16671875" width="0.254" layer="1"/>
@@
 <via x="40.6908" y="6.1722" extent="1-16" drill="0.6096"/>
 <via x="29.9466" y="10.5156" extent="1-16" drill="0.6096"/>
+<wire x1="49.443640625" y1="10.149840625" x2="49.443640625" y2="9.51991875" width="0.254" layer="1"/>
+<wire x1="49.443640625" y1="9.51991875" x2="50.886359375" y2="8.0772" width="0.254" layer="1"/>
+<wire x1="50.886359375" y1="8.0772" x2="51.4959625" y2="8.0772" width="0.254" layer="1"/>
+<wire x1="51.4959625" y1="8.0772" x2="51.506121875" y2="8.087359375" width="0.254" layer="1"/>
 </signal>
 <signal name="IO4">
@@
 <wire x1="52.743996875" y1="2.6771625" x2="52.743996875" y2="6.32968125" width="0.254" layer="1"/>
 <wire x1="52.743996875" y1="6.32968125" x2="52.633878125" y2="6.32968125" width="0.254" layer="1"/>
-<wire x1="52.633878125" y1="6.32968125" x2="50.4952" y2="8.468359375" width="0.254" layer="1"/>
-<wire x1="50.4952" y1="8.468359375" x2="48.337840625" y2="8.468359375" width="0.254" layer="1"/>
 <wire x1="48.337840625" y1="8.468359375" x2="48.3362" y2="8.46671875" width="0.254" layer="1"/>
 <wire x1="48.3362" y1="8.46671875" x2="44.46524375" y2="8.46671875" width="0.254" layer="1"/>
@@
 <wire x1="10.33271875" y1="8.315959375" x2="15.001240625" y2="8.315959375" width="0.254" layer="16"/>
 <wire x1="15.001240625" y1="8.315959375" x2="15.5448" y2="7.7724" width="0.254" layer="16"/>
-<polygon width="0.254" layer="1">
+<polygon width="0.0254" layer="1">
 <vertex x="-2.550159375" y="33.004759375"/>
 <vertex x="-3.20548125" y="33.004759375"/>
@@
 <vertex x="-1.153159375" y="33.25368125"/>
 </polygon>
-<polygon width="0.254" layer="16">
+<polygon width="0.0254" layer="16">
 <vertex x="-2.87528125" y="-13.578840625"/>
 <vertex x="69.22008125" y="-13.578840625"/>
@@
 <via x="24.038559375" y="6.832596875" extent="1-16" drill="0.6"/>
 <via x="42.6618375" y="6.761478125" extent="1-16" drill="0.6"/>
-<via x="34.701478125" y="9.4996" extent="1-16" drill="0.6"/>
-<via x="41.402" y="8.031478125" extent="1-16" drill="0.6"/>
+<via x="34.676078125" y="9.59611875" extent="1-16" drill="0.6"/>
+<via x="41.341040625" y="8.14831875" extent="1-16" drill="0.6"/>
 </signal>
 <signal name="OUTL">
@@
 <contactref element="R5" pad="2"/>
 <contactref element="U$1" pad="17"/>
-<wire x1="37.090953125" y1="8.8083625" x2="41.000321875" y2="8.8083625" width="0.254" layer="1"/>
-<wire x1="41.000321875" y1="8.8083625" x2="41.310559375" y2="9.1186" width="0.254" layer="1"/>
 <wire x1="41.310559375" y1="9.1186" x2="41.310559375" y2="9.746871875" width="0.254" layer="1"/>
 <wire x1="41.310559375" y1="9.746871875" x2="41.347759375" y2="9.784071875" width="0.254" layer="1"/>
-<wire x1="37.090953125" y1="8.8083625" x2="38.979196875" y2="8.8083625" width="0.254" layer="1"/>
-<wire x1="38.979196875" y1="8.8083625" x2="39.72051875" y2="8.067040625" width="0.254" layer="1"/>
 <wire x1="39.72051875" y1="8.067040625" x2="39.72051875" y2="3.623671875" width="0.254" layer="1"/>
 <wire x1="39.72051875" y1="3.623671875" x2="39.698565625" y2="3.60171875" width="0.254" layer="1"/>
+<wire x1="39.72051875" y1="8.067040625" x2="38.4200375" y2="8.067040625" width="0.254" layer="1"/>
+<wire x1="38.4200375" y1="8.067040625" x2="37.678359375" y2="8.80871875" width="0.254" layer="1"/>
+<wire x1="37.678359375" y1="8.80871875" x2="37.091309375" y2="8.80871875" width="0.254" layer="1"/>
+<wire x1="37.091309375" y1="8.80871875" x2="37.090953125" y2="8.8083625" width="0.254" layer="1"/>
+<wire x1="39.72051875" y1="8.067040625" x2="40.259" y2="8.067040625" width="0.254" layer="1"/>
+<wire x1="41.310559375" y1="9.1186" x2="40.833040625" y2="9.1186" width="0.254" layer="1"/>
+<wire x1="40.833040625" y1="9.1186" x2="40.4368" y2="8.722359375" width="0.254" layer="1"/>
+<wire x1="40.4368" y1="8.722359375" x2="40.4368" y2="8.244840625" width="0.254" layer="1"/>
+<wire x1="40.4368" y1="8.244840625" x2="40.259" y2="8.067040625" width="0.254" layer="1"/>
 </signal>
 <signal name="N$4">
@@
 <contactref element="C2" pad="1"/>
 <wire x1="37.090953125" y1="9.4583625" x2="38.23775625" y2="9.4583625" width="0.254" layer="1"/>
-<wire x1="38.23775625" y1="9.4583625" x2="38.24731875" y2="9.4488" width="0.254" layer="1"/>
-<via x="38.24731875" y="9.4488" extent="1-16" drill="0.6"/>
-<wire x1="38.24731875" y1="9.4488" x2="41.402" y2="9.4488" width="0.254" layer="16"/>
+<wire x1="38.23775625" y1="9.4583625" x2="38.29811875" y2="9.4488" width="0.254" layer="1"/>
+<via x="38.29811875" y="9.4488" extent="1-16" drill="0.6"/>
+<wire x1="38.29811875" y1="9.4488" x2="41.402" y2="9.4488" width="0.254" layer="16"/>
 <wire x1="41.402" y1="9.4488" x2="44.54651875" y2="6.30428125" width="0.254" layer="16"/>
 <wire x1="44.54651875" y1="6.30428125" x2="47.1525625" y2="6.30428125" width="0.254" layer="16"/>
