File: Odroid Headphone Hat.sch (EAGLE design)
At the start: 20 parts, among them X1 1501_03, X2 1501_03

Commit message: A few tweeks
Changed lines of the file:
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@@
 <wire x1="187.96" y1="78.74" x2="203.2" y2="78.74" width="0.1524" layer="91"/>
 <label x="193.04" y="78.74" size="1.778" layer="95"/>
+<junction x="187.96" y="78.74"/>
 </segment>
 <segment>
@@
 </sheet>
 </sheets>
+<errors>
+</errors>
 </schematic>
 </drawing>

Commit message: tweeks to get working - no headphone mod yet
Parts:
- C8, C9: value 2u2 -> 2n2
- R1: value 7k5 -> 2k7
- R5: value 2k7 -> 7k5
Changed lines of the file:
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@@
 <part name="JP1" library="pinhead" deviceset="PINHD-1X10" device="/90"/>
 <part name="C1" library="resistor" deviceset="C-EU" device="C0603" value="100nF"/>
-<part name="R1" library="resistor" deviceset="R-EU_" device="R0603" value="7k5"/>
+<part name="R1" library="resistor" deviceset="R-EU_" device="R0603" value="2k7"/>
 <part name="R2" library="resistor" deviceset="R-EU_" device="R0603" value="22R"/>
 <part name="R3" library="resistor" deviceset="R-EU_" device="R0603" value="22R"/>
 <part name="R4" library="resistor" deviceset="R-EU_" device="R0603" value="22R"/>
 <part name="C2" library="resistor" deviceset="C-EU" device="C0603" value="100nF"/>
-<part name="R5" library="resistor" deviceset="R-EU_" device="R0603" value="2k7"/>
+<part name="R5" library="resistor" deviceset="R-EU_" device="R0603" value="7k5"/>
 <part name="C3" library="resistor" deviceset="C-EU" device="C0603" value="2u2"/>
 <part name="C4" library="resistor" deviceset="C-EU" device="C0603" value="2u2"/>
@@
 <part name="R6" library="resistor" deviceset="R-EU_" device="R0603" value="470R"/>
 <part name="R7" library="resistor" deviceset="R-EU_" device="R0603" value="470R"/>
-<part name="C8" library="resistor" deviceset="C-EU" device="C0603" value="2u2"/>
-<part name="C9" library="resistor" deviceset="C-EU" device="C0603" value="2u2"/>
+<part name="C8" library="resistor" deviceset="C-EU" device="C0603" value="2n2"/>
+<part name="C9" library="resistor" deviceset="C-EU" device="C0603" value="2n2"/>
 <part name="X2" library="con-lumberg" deviceset="1501_03" device=""/>
 <part name="X1" library="con-lumberg" deviceset="1501_03" device=""/>
